File: 50x50_2x6_to_sma.sch (KiCad schematic (older format))
At the start: 17 parts, among them J1 Conn_Coaxial, J10 Conn_Coaxial, J11 Conn_Coaxial, J12 Conn_Coaxial, J2 Conn_Coaxial, J20 Conn_02x06_Counter_Clockwise, J21 Conn_01x06, J22 Conn_01x06, J23 Conn_01x06, J24 Conn_01x06, J3 Conn_Coaxial, J4 Conn_Coaxial, J5 Conn_Coaxial, J6 Conn_Coaxial, J7 Conn_Coaxial, J8 Conn_Coaxial, J9 Conn_Coaxial

Commit message: Add pin header library
Parts:
- J1, J10, J11, J12, J2, J3, J4, J5, J6, J7, J8, J9: footprint (none) -> Connectors:SMA_Board_Edge
- J20: footprint (none) -> Pin_Headers:Pin_Header_Straight_2x06_Pitch2.54mm; symbol Conn_02x06_Counter_Clockwise -> Conn_02x06_Odd_Even
- J21, J22: footprint (none) -> Pin_Headers:Pin_Header_Straight_1x06_Pitch2.54mm
- J23, J24: footprint (none) -> 2.54mm_Pin_Headers:Edge_1x06
Connections:
- net GND: now also J1.2 (Ext), J10.2 (Ext), J11.2 (Ext), J12.2 (Ext), J2.2 (Ext), J23.1 (Pin_1), J23.2 (Pin_2), J23.3 (Pin_3), J23.4 (Pin_4), J23.5 (Pin_5), J23.6 (Pin_6), J24.1 (Pin_1), J24.2 (Pin_2), J24.3 (Pin_3), J24.4 (Pin_4), J24.5 (Pin_5), J24.6 (Pin_6), J3.2 (Ext), J4.2 (Ext), J5.2 (Ext), J6.2 (Ext), J7.2 (Ext), J8.2 (Ext), J9.2 (Ext)
- net at J20.12 (Pin_12), J22.6 (Pin_6): now also J7.1 (In); no longer J12.1 (In)
- net at J2.1 (In), J21.2 (Pin_2): now also J20.3 (Pin_3); no longer J20.2 (Pin_2)
- net at J21.3 (Pin_3), J3.1 (In): now also J20.5 (Pin_5); no longer J20.3 (Pin_3)
- net at J21.4 (Pin_4), J4.1 (In): now also J20.7 (Pin_7); no longer J20.4 (Pin_4)
- net at J21.5 (Pin_5), J5.1 (In): now also J20.9 (Pin_9); no longer J20.5 (Pin_5)
- net at J21.6 (Pin_6), J6.1 (In): now also J20.11 (Pin_11); no longer J20.6 (Pin_6)
- new net: J20.10 (Pin_10), J22.5 (Pin_5), J8.1 (In)
- new net: J12.1 (In), J20.2 (Pin_2), J22.1 (Pin_1)
- new net: J11.1 (In), J20.4 (Pin_4), J22.2 (Pin_2)
- new net: J10.1 (In), J20.6 (Pin_6), J22.3 (Pin_3)
- new net: J20.8 (Pin_8), J22.4 (Pin_4), J9.1 (In)
Changed lines of the file:
@@
 $EndDescr
 $Comp
-L Conn_02x06_Counter_Clockwise J20
+L Conn_02x06_Odd_Even J20
 U 1 1 59C0351E
 P 1600 1550
 F 0 "J20" H 1650 1850 50  0000 C CNN
 F 1 "Conn_02x06_Counter_Clockwise" H 1650 1150 50  0001 C CNN
-F 2 "" H 1600 1550 50  0001 C CNN
+F 2 "Pin_Headers:Pin_Header_Straight_2x06_Pitch2.54mm" H 1600 1550 50  0001 C CNN
 F 3 "" H 1600 1550 50  0001 C CNN
 	1    1600 1550
@@
 F 0 "J21" H 1200 1850 50  0000 C CNN
 F 1 "Conn_01x06" H 1200 1150 50  0001 C CNN
-F 2 "" H 1200 1550 50  0001 C CNN
+F 2 "Pin_Headers:Pin_Header_Straight_1x06_Pitch2.54mm" H 1200 1550 50  0001 C CNN
 F 3 "" H 1200 1550 50  0001 C CNN
 	1    1200 1550
 	-1   0    0    -1
-$EndComp
-$Comp
-L Conn_01x06 J22
-U 1 1 59C03686
-P 2100 1650
-F 0 "J22" H 2100 1250 50  0000 C CNN
-F 1 "Conn_01x06" H 2100 1250 50  0001 C CNN
-F 2 "" H 2100 1650 50  0001 C CNN
-F 3 "" H 2100 1650 50  0001 C CNN
-	1    2100 1650
-	1    0    0    1
 $EndComp
 $Comp
@@
 F 0 "J2" H 650 750 50  0000 C CNN
 F 1 "Conn_Coaxial" V 865 800 50  0001 C CNN
-F 2 "" H 750 800 50  0001 C CNN
+F 2 "Connectors:SMA_Board_Edge" H 750 800 50  0001 C CNN
 F 3 "" H 750 800 50  0001 C CNN
 	1    750  800
@@
 F 0 "J11" H 2450 750 50  0000 C CNN
 F 1 "Conn_Coaxial" V 2665 800 50  0001 C CNN
-F 2 "" H 2550 800 50  0001 C CNN
+F 2 "Connectors:SMA_Board_Edge" H 2550 800 50  0001 C CNN
 F 3 "" H 2550 800 50  0001 C CNN
 	1    2550 800
@@
 F 0 "J8" H 2400 2500 50  0000 C CNN
 F 1 "Conn_Coaxial" V 2665 2450 50  0001 C CNN
-F 2 "" H 2550 2450 50  0001 C CNN
+F 2 "Connectors:SMA_Board_Edge" H 2550 2450 50  0001 C CNN
 F 3 "" H 2550 2450 50  0001 C CNN
 	1    2550 2450
@@
 F 0 "J5" H 600 2500 50  0000 C CNN
 F 1 "Conn_Coaxial" V 865 2450 50  0001 C CNN
-F 2 "" H 750 2450 50  0001 C CNN
+F 2 "Connectors:SMA_Board_Edge" H 750 2450 50  0001 C CNN
 F 3 "" H 750 2450 50  0001 C CNN
 	1    750  2450
@@
 F 0 "J6" V 1450 2500 50  0000 C CNN
 F 1 "Conn_Coaxial" V 1665 2450 50  0001 C CNN
-F 2 "" H 1550 2450 50  0001 C CNN
+F 2 "Connectors:SMA_Board_Edge" H 1550 2450 50  0001 C CNN
 F 3 "" H 1550 2450 50  0001 C CNN
 	1    1550 2450
@@
 F 0 "J7" V 1650 2400 50  0000 C CNN
 F 1 "Conn_Coaxial" V 1865 2450 50  0001 C CNN
-F 2 "" H 1750 2450 50  0001 C CNN
+F 2 "Connectors:SMA_Board_Edge" H 1750 2450 50  0001 C CNN
 F 3 "" H 1750 2450 50  0001 C CNN
 	1    1750 2450
@@
 F 0 "J3" H 650 1550 50  0000 C CNN
 F 1 "Conn_Coaxial" V 865 1500 50  0001 C CNN
-F 2 "" H 750 1500 50  0001 C CNN
+F 2 "Connectors:SMA_Board_Edge" H 750 1500 50  0001 C CNN
 F 3 "" H 750 1500 50  0001 C CNN
 	1    750  1500
@@
 F 0 "J4" H 650 1650 50  0000 C CNN
 F 1 "Conn_Coaxial" V 865 1700 50  0001 C CNN
-F 2 "" H 750 1700 50  0001 C CNN
+F 2 "Connectors:SMA_Board_Edge" H 750 1700 50  0001 C CNN
 F 3 "" H 750 1700 50  0001 C CNN
 	1    750  1700
@@
 F 0 "J9" H 2400 1650 50  0000 C CNN
 F 1 "Conn_Coaxial" V 2665 1700 50  0001 C CNN
-F 2 "" H 2550 1700 50  0001 C CNN
+F 2 "Connectors:SMA_Board_Edge" H 2550 1700 50  0001 C CNN
 F 3 "" H 2550 1700 50  0001 C CNN
 	1    2550 1700
@@
 F 0 "J10" H 2400 1450 50  0000 C CNN
 F 1 "Conn_Coaxial" V 2665 1500 50  0001 C CNN
-F 2 "" H 2550 1500 50  0001 C CNN
+F 2 "Connectors:SMA_Board_Edge" H 2550 1500 50  0001 C CNN
 F 3 "" H 2550 1500 50  0001 C CNN
 	1    2550 1500
@@
 F 0 "J12" V 1650 700 50  0000 C CNN
 F 1 "Conn_Coaxial" V 1865 800 50  0001 C CNN
-F 2 "" H 1750 800 50  0001 C CNN
+F 2 "Connectors:SMA_Board_Edge" H 1750 800 50  0001 C CNN
 F 3 "" H 1750 800 50  0001 C CNN
 	1    1750 800
@@
 F 0 "J1" V 1450 850 50  0000 C CNN
 F 1 "Conn_Coaxial" V 1665 800 50  0001 C CNN
-F 2 "" H 1550 800 50  0001 C CNN
+F 2 "Connectors:SMA_Board_Edge" H 1550 800 50  0001 C CNN
 F 3 "" H 1550 800 50  0001 C CNN
 	1    1550 800
@@
 F 0 "J23" H 1250 3250 50  0000 C CNN
 F 1 "Conn_01x06" H 1250 2550 50  0001 C CNN
-F 2 "" H 1250 2950 50  0001 C CNN
+F 2 "2.54mm_Pin_Headers:Edge_1x06" H 1250 2950 50  0001 C CNN
 F 3 "" H 1250 2950 50  0001 C CNN
 	1    1250 2950
@@
 F 0 "J24" H 2150 3250 50  0000 C CNN
 F 1 "Conn_01x06" H 2150 2550 50  0001 C CNN
-F 2 "" H 2150 2950 50  0001 C CNN
+F 2 "2.54mm_Pin_Headers:Edge_1x06" H 2150 2950 50  0001 C CNN
 F 3 "" H 2150 2950 50  0001 C CNN
 	1    2150 2950
@@
 	2350 2750 2350 2650
 Connection ~ 2350 2650
+$Comp
+L Conn_01x06 J22
+U 1 1 59C03686
+P 2100 1550
+F 0 "J22" H 2100 1850 50  0000 C CNN
+F 1 "Conn_01x06" H 2100 1150 50  0001 C CNN
+F 2 "Pin_Headers:Pin_Header_Straight_1x06_Pitch2.54mm" H 2100 1550 50  0001 C CNN
+F 3 "" H 2100 1550 50  0001 C CNN
+	1    2100 1550
+	1    0    0    -1
+$EndComp
+Text Label 1550 2650 0    60   ~ 0
+GND
 $EndSCHEMATC
